Commit message: URDF changes

File: TestContainer/HumbleGazebo/SimulationFiles/install/robot_desc/share/robot_desc/robot/robot.urdf (robot description, URDF)
Before this commit: robot project_robot, 1 links, 0 joints
Links:
- link part_1: mass 1e-09 -> 0.117967; geometry collision mesh filename=package://robot_desc/robot/assets/8020_1530_x_48.stl; collision mesh filename=package://robot_desc/robot/assets/armbasemount.stl

Commit message: urdf

File: TestContainer/HumbleGazebo/SimulationFiles/install/robot_desc/share/robot_desc/robot/robot.urdf (robot description, URDF)
Before this commit: robot project_robot, 1 links, 0 joints
Links:
- removed link part_1
- added link EEframe, mass 1e-9
- added link armbasemount, mass 0.0616; collision mesh filename=robot_desc/robot/assets/armbasemount.stl; visual mesh filename=robot_desc/robot/assets/armbasemount.stl
- added link combinedshoulder, mass 0.0159914; collision mesh filename=robot_desc/robot/assets/combinedshoulder.stl; visual mesh filename=robot_desc/robot/assets/combinedshoulder.stl
- added link dynamixelmotor_withhorn, mass 0.0822187; collision mesh filename=robot_desc/robot/assets/dynamixelmotor_withhorn.stl; visual mesh filename=robot_desc/robot/assets/dynamixelmotor_withhorn.stl
- added link dynamixelmotor_withhorn_2, mass 0.0822187; collision mesh filename=robot_desc/robot/assets/dynamixelmotor_withhorn.stl; visual mesh filename=robot_desc/robot/assets/dynamixelmotor_withhorn.stl
- added link hooplink, mass 0.0174; collision mesh filename=robot_desc/robot/assets/hooplink.stl; visual mesh filename=robot_desc/robot/assets/hooplink.stl
Joints:
- added joint EEframe_frame: type fixed, parent hooplink, child EEframe, origin xyz=0.3 -0.0002 0.003 rpy=0 -0 2.97496e-65, axis 0 0 0
- added joint elbow: type revolute, parent dynamixelmotor_withhorn_2, child hooplink, origin xyz=0.0358 0.0085 0.0055 rpy=-1.71531e-32 1.36846e-48 2.42861e-17, axis 0 0 1, limit lower=-2.30383 upper=2.30383 effort=10 velocity=10
- added joint elbowmotor: type fixed, parent combinedshoulder, child dynamixelmotor_withhorn_2, origin xyz=0.2622 0.0085 0 rpy=-3.14159 -0 -2.97496e-65, axis 0 0 1, limit effort=10 velocity=10
- added joint shoulder: type revolute, parent dynamixelmotor_withhorn, child combinedshoulder, origin xyz=-0.0358 -0.0085 0.00548 rpy=-3.14159 1.2326e-32 3.13167, axis 0 0 1, limit lower=-1.58072 upper=1.56087 effort=10 velocity=10
- added joint shouldermotor: type fixed, parent armbasemount, child dynamixelmotor_withhorn, origin xyz=0.0085 0.0678 0.09305 rpy=0 -0 -1.5708, axis 0 0 1, limit effort=10 velocity=10

File: TestContainer/HumbleGazebo/SimulationFiles/src/robot_desc/robot/robot.urdf (robot description, URDF)
Before this commit: robot project_robot, 4 links, 3 joints
Links:
- added link combinedshoulder, mass 0.0159914; collision mesh filename=robot_desc/robot/assets/combinedshoulder.stl; visual mesh filename=robot_desc/robot/assets/combinedshoulder.stl
- added link dynamixelmotor_withhorn_2, mass 0.0822187; collision mesh filename=robot_desc/robot/assets/dynamixelmotor_withhorn.stl; visual mesh filename=robot_desc/robot/assets/dynamixelmotor_withhorn.stl
- link armbasemount: mass 0.143819 -> 0.0616; geometry collision mesh filename=robot_desc/robot/assets/armbasemount.stl; visual mesh filename=robot_desc/robot/assets/armbasemount.stl
- link dynamixelmotor_withhorn: mass 0.0982101 -> 0.0822187; geometry collision mesh filename=robot_desc/robot/assets/dynamixelmotor_withhorn.stl; visual mesh filename=robot_desc/robot/assets/dynamixelmotor_withhorn.stl
- link hooplink: geometry collision mesh filename=robot_desc/robot/assets/hooplink.stl; visual mesh filename=robot_desc/robot/assets/hooplink.stl
Joints:
- added joint elbowmotor: type fixed, parent combinedshoulder, child dynamixelmotor_withhorn_2, origin xyz=0.2622 0.0085 0 rpy=-3.14159 -0 -2.97496e-65, axis 0 0 1, limit effort=10 velocity=10
- added joint shouldermotor: type fixed, parent armbasemount, child dynamixelmotor_withhorn, origin xyz=0.0085 0.0678 0.09305 rpy=0 -0 -1.5708, axis 0 0 1, limit effort=10 velocity=10
- joint elbow: origin xyz=0.298 3.3632e-16 -0.0055 rpy=3.14159 -1.36846e-48 -2.42861e-17 -> xyz=0.0358 0.0085 0.0055 rpy=-1.71531e-32 1.36846e-48 2.42861e-17; parent dynamixelmotor_withhorn -> dynamixelmotor_withhorn_2
- joint shoulder: child dynamixelmotor_withhorn -> combinedshoulder; origin xyz=-1.43115e-17 0.1036 0.09853 rpy=-3.14159 1.2326e-32 1.56087 -> xyz=-0.0358 -0.0085 0.00548 rpy=-3.14159 1.2326e-32 3.13167; parent armbasemount -> dynamixelmotor_withhorn

Commit message: Start publisher node for RViz

File: TestContainer/HumbleGazebo/SimulationFiles/install/robot_desc/share/robot_desc/robot/robot.urdf (robot description, URDF)
Before this commit: robot project_robot, 6 links, 5 joints
Links:
- link armbasemount: geometry collision mesh filename=package://robot_desc/robot/assets/armbasemount.stl; visual mesh filename=package://robot_desc/robot/assets/armbasemount.stl
- link combinedshoulder: geometry collision mesh filename=package://robot_desc/robot/assets/combinedshoulder.stl; visual mesh filename=package://robot_desc/robot/assets/combinedshoulder.stl
- link dynamixelmotor_withhorn: geometry collision mesh filename=package://robot_desc/robot/assets/dynamixelmotor_withhorn.s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; visual mesh filename=package://robot_desc/robot/assets/dynamixelmotor_withhorn.s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
- link dynamixelmotor_withhorn_2: geometry collision mesh filename=package://robot_desc/robot/assets/dynamixelmotor_withhorn.s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; visual mesh filename=package://robot_desc/robot/assets/dynamixelmotor_withhorn.s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
- link hooplink: geometry collision mesh filename=package://robot_desc/robot/assets/hooplink.stl; visual mesh filename=package://robot_desc/robot/assets/hooplink.stl
